File: hardware/playa.brd (EAGLE design)
At the start: 70 x 65 mm, 89 parts, among them Q2 12.288MHz, Q3 8MHz, U1 ATMEGA328, U11 1.8v, U12 3.3v, U17 AVR_SPI_PRG_6PTH, U3 microSD Socket, U5 3.3v, U6 CN3083, U9 VS1053-L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

Commit message: modify battery voltage divider. it currently uses 35uA
Parts:
- R19: value 2M 1% -> 68k 1%
- R8: value 10M 1% -> 39k 1%
Changed lines of the file:
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@@
 <element name="U$3" library="tsop" package="TSOP312X" value="TSOP312X" x="61.8" y="53.8" rot="R180"/>
 <element name="C11" library="rcl" package="C1206" value="4.7u" x="57.2" y="58.2" rot="R180"/>
-<element name="R8" library="rcl" package="R0805W" value="10M 1%" x="47.8" y="9" rot="R90"/>
-<element name="R19" library="rcl" package="R0805W" value="2M 1%" x="46.8" y="13.2" rot="R180"/>
+<element name="R8" library="rcl" package="R0805W" value="39k 1%" x="47.8" y="9" rot="R90"/>
+<element name="R19" library="rcl" package="R0805W" value="68k 1%" x="46.8" y="13.2" rot="R180"/>
 <element name="C17" library="rcl" package="C0805" value="100nF" x="50.4" y="9" rot="R270"/>
 <element name="U$5" library="SparkFun" package="OSHW-LOGO-M" value="OSHW-LOGOM" x="15.4" y="43.2"/>

Commit message: rename traces to match the names given in the source code
Connections:
- net O_DETECT renamed JACK_DETECT
- net VIN_DETECT renamed VBAT_DETECT
Changed lines of the file:
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@@
 <?xml version="1.0" encoding="utf-8"?>
 <!DOCTYPE eagle SYSTEM "eagle.dtd">
-<eagle version="6.1">
+<eagle version="6.4">
 <drawing>
 <settings>
@@
 <layer number="23" name="tOrigins" color="15" fill="1" visible="yes" active="yes"/>
 <layer number="24" name="bOrigins" color="15" fill="1" visible="yes" active="yes"/>
-<layer number="25" name="tNames" color="7" fill="1" visible="no" active="yes"/>
-<layer number="26" name="bNames" color="7" fill="1" visible="no" active="yes"/>
-<layer number="27" name="tValues" color="7" fill="1" visible="no" active="yes"/>
-<layer number="28" name="bValues" color="7" fill="1" visible="no" active="yes"/>
+<layer number="25" name="tNames" color="7" fill="1" visible="yes" active="yes"/>
+<layer number="26" name="bNames" color="7" fill="1" visible="yes" active="yes"/>
+<layer number="27" name="tValues" color="7" fill="1" visible="yes" active="yes"/>
+<layer number="28" name="bValues" color="7" fill="1" visible="yes" active="yes"/>
 <layer number="29" name="tStop" color="7" fill="3" visible="no" active="yes"/>
 <layer number="30" name="bStop" color="7" fill="6" visible="no" active="yes"/>
-<layer number="31" name="tCream" color="7" fill="4" visible="yes" active="yes"/>
-<layer number="32" name="bCream" color="7" fill="5" visible="yes" active="yes"/>
-<layer number="33" name="tFinish" color="6" fill="3" visible="yes" active="yes"/>
-<layer number="34" name="bFinish" color="6" fill="6" visible="yes" active="yes"/>
-<layer number="35" name="tGlue" color="7" fill="4" visible="yes" active="yes"/>
-<layer number="36" name="bGlue" color="7" fill="5" visible="yes" active="yes"/>
+<layer number="31" name="tCream" color="7" fill="4" visible="no" active="yes"/>
+<layer number="32" name="bCream" color="7" fill="5" visible="no" active="yes"/>
+<layer number="33" name="tFinish" color="6" fill="3" visible="no" active="yes"/>
+<layer number="34" name="bFinish" color="6" fill="6" visible="no" active="yes"/>
+<layer number="35" name="tGlue" color="7" fill="4" visible="no" active="yes"/>
+<layer number="36" name="bGlue" color="7" fill="5" visible="no" active="yes"/>
 <layer number="37" name="tTest" color="7" fill="1" visible="yes" active="yes"/>
 <layer number="38" name="bTest" color="7" fill="1" visible="yes" active="yes"/>
@@
 </class>
 </classes>
-<designrules>
+<designrules name="default">
 <description language="de">&lt;b&gt;EAGLE Design Rules&lt;/b&gt;
 &lt;p&gt;
@@
 <wire x1="5" y1="43" x2="7" y2="45" width="0.6096" layer="1"/>
 </signal>
-<signal name="O_DETECT">
-<contactref element="U1" pad="24"/>
-<contactref element="R24" pad="1"/>
-<contactref element="X2" pad="B"/>
-<wire x1="46.6" y1="44.7074" x2="46.6" y2="43.6" width="0.4064" layer="1"/>
-<wire x1="7" y1="49.3" x2="7" y2="56.6" width="0.6096" layer="16"/>
-<wire x1="47.8" y1="54.2" x2="47.8" y2="44.8" width="0.4064" layer="16"/>
-<wire x1="48.8" y1="54.6" x2="47.8" y2="54.2" width="0.4064" layer="16"/>
-<wire x1="47.8" y1="44.8" x2="47.8" y2="42.46" width="0.4064" layer="1"/>
-<wire x1="47.8" y1="42.46" x2="48.06" y2="42.2" width="0.4064" layer="1"/>
-<wire x1="46.6" y1="42.6" x2="46.6" y2="44.7074" width="0.4064" layer="1"/>
-<wire x1="47" y1="42.2" x2="46.6" y2="42.6" width="0.4064" layer="1"/>
-<wire x1="48.06" y1="42.2" x2="47" y2="42.2" width="0.4064" layer="1"/>
-<wire x1="48" y1="60" x2="48" y2="56" width="0.4064" layer="1"/>
-<wire x1="48" y1="56" x2="48.8" y2="55.2" width="0.4064" layer="1"/>
-<wire x1="48.8" y1="55.2" x2="48.8" y2="54.6" width="0.4064" layer="1"/>
-<wire x1="47.2" y1="61.4" x2="48" y2="60.6" width="0.4064" layer="16"/>
-<wire x1="48" y1="60.6" x2="48" y2="60" width="0.4064" layer="16"/>
-<wire x1="7" y1="56.6" x2="7" y2="57.6" width="0.4064" layer="16"/>
-<wire x1="8.1" y1="48.2" x2="7" y2="49.3" width="0.6096" layer="16"/>
-<wire x1="8.7" y1="48.2" x2="8.1" y2="48.2" width="0.6096" layer="16"/>
-<wire x1="7" y1="57.6" x2="8.6" y2="59.2" width="0.4064" layer="16"/>
-<wire x1="8.6" y1="59.2" x2="8.6" y2="60.4" width="0.4064" layer="16"/>
-<wire x1="8.6" y1="60.4" x2="9.6" y2="61.4" width="0.4064" layer="16"/>
-<wire x1="9.6" y1="61.4" x2="47.2" y2="61.4" width="0.4064" layer="16"/>
-<via x="47.8" y="44.8" extent="1-16" drill="0.5"/>
-<via x="48" y="60" extent="1-16" drill="0.4"/>
-<via x="48.8" y="54.6" extent="1-16" drill="0.4"/>
-</signal>
 <signal name="N$17">
 <contactref element="U9" pad="36"/>
@@
 <wire x1="59.26" y1="53.8" x2="58.6" y2="54.46" width="0.6096" layer="1"/>
 </signal>
-<signal name="VIN_DETECT">
-<contactref element="R8" pad="2"/>
-<contactref element="R19" pad="1"/>
-<contactref element="C17" pad="1"/>
-<contactref element="U1" pad="28"/>
-<wire x1="47.8" y1="9.94" x2="47.8" y2="10.6" width="0.4064" layer="1"/>
-<wire x1="47.8" y1="10.6" x2="47.8" y2="13.14" width="0.3048" layer="1"/>
-<wire x1="47.8" y1="13.14" x2="47.74" y2="13.2" width="0.4064" layer="1"/>
-<wire x1="48.2" y1="10.2" x2="50.4" y2="10.2" width="0.3048" layer="1"/>
-<wire x1="50.4" y1="10.2" x2="61.8" y2="10.2" width="0.3048" layer="1"/>
-<wire x1="47.8" y1="10.6" x2="48.2" y2="10.2" width="0.4064" layer="1"/>
-<wire x1="61.8" y1="10.2" x2="61.8" y2="16.2" width="0.3048" layer="16"/>
-<wire x1="50.4" y1="10.2" x2="50.4" y2="9.85" width="0.3048" layer="1"/>
-<wire x1="50.2" y1="48.6" x2="48.0926" y2="48.6" width="0.3048" layer="1"/>
-<wire x1="52.4" y1="46.4" x2="50.2" y2="48.6" width="0.3048" layer="1"/>
-<wire x1="60.8" y1="46.4" x2="52.4" y2="46.4" width="0.3048" layer="1"/>
-<wire x1="61.8" y1="45.4" x2="60.8" y2="46.4" width="0.3048" layer="1"/>
-<wire x1="61.8" y1="16.2" x2="61.8" y2="45.4" width="0.3048" layer="1"/>
-<via x="61.8" y="10.2" extent="1-16" drill="0.5"/>
-<via x="61.8" y="16.2" extent="1-16" drill="0.5"/>
-</signal>
 <signal name="SW1">
 <contactref element="U1" pad="27"/>
@@
 <wire x1="59.4" y1="34.2" x2="59.4" y2="43.4" width="0.3048" layer="1"/>
 </signal>
+<signal name="JACK_DETECT">
+<contactref element="U1" pad="24"/>
+<contactref element="R24" pad="1"/>
+<wire x1="46.6" y1="44.7074" x2="46.6" y2="43.6" width="0.4064" layer="1"/>
+<wire x1="46.6" y1="42.6" x2="46.6" y2="44.7074" width="0.4064" layer="1"/>
+<wire x1="47" y1="42.2" x2="46.6" y2="42.6" width="0.4064" layer="1"/>
+<wire x1="48.06" y1="42.2" x2="47" y2="42.2" width="0.4064" layer="1"/>
+<contactref element="X2" pad="B"/>
+<wire x1="7" y1="49.3" x2="7" y2="56.6" width="0.6096" layer="16"/>
+<wire x1="47.8" y1="54.2" x2="47.8" y2="44.8" width="0.4064" layer="16"/>
+<wire x1="48.8" y1="54.6" x2="47.8" y2="54.2" width="0.4064" layer="16"/>
+<wire x1="47.8" y1="44.8" x2="47.8" y2="42.2" width="0.4064" layer="1"/>
+<wire x1="48" y1="60" x2="48" y2="56" width="0.4064" layer="1"/>
+<wire x1="48" y1="56" x2="48.8" y2="55.2" width="0.4064" layer="1"/>
+<wire x1="48.8" y1="55.2" x2="48.8" y2="54.6" width="0.4064" layer="1"/>
+<wire x1="47.2" y1="61.4" x2="48" y2="60.6" width="0.4064" layer="16"/>
+<wire x1="48" y1="60.6" x2="48" y2="60" width="0.4064" layer="16"/>
+<wire x1="7" y1="56.6" x2="7" y2="57.6" width="0.4064" layer="16"/>
+<wire x1="8.1" y1="48.2" x2="7" y2="49.3" width="0.6096" layer="16"/>
+<wire x1="8.7" y1="48.2" x2="8.1" y2="48.2" width="0.6096" layer="16"/>
+<wire x1="7" y1="57.6" x2="8.6" y2="59.2" width="0.4064" layer="16"/>
+<wire x1="8.6" y1="59.2" x2="8.6" y2="60.4" width="0.4064" layer="16"/>
+<wire x1="8.6" y1="60.4" x2="9.6" y2="61.4" width="0.4064" layer="16"/>
+<wire x1="9.6" y1="61.4" x2="47.2" y2="61.4" width="0.4064" layer="16"/>
+<via x="47.8" y="44.8" extent="1-16" drill="0.5"/>
+<via x="48" y="60" extent="1-16" drill="0.4"/>
+<via x="48.8" y="54.6" extent="1-16" drill="0.4"/>
+<wire x1="48.06" y1="42.2" x2="47.8" y2="42.2" width="0.4064" layer="1"/>
+</signal>
+<signal name="VBAT_DETECT">
+<contactref element="U1" pad="28"/>
+<contactref element="R8" pad="2"/>
+<contactref element="R19" pad="1"/>
+<contactref element="C17" pad="1"/>
+<wire x1="47.8" y1="9.94" x2="47.8" y2="10.6" width="0.4064" layer="1"/>
+<wire x1="47.8" y1="10.6" x2="47.8" y2="13.14" width="0.3048" layer="1"/>
+<wire x1="47.8" y1="13.14" x2="47.74" y2="13.2" width="0.4064" layer="1"/>
+<wire x1="48.2" y1="10.2" x2="50.4" y2="10.2" width="0.3048" layer="1"/>
+<wire x1="50.4" y1="10.2" x2="61.8" y2="10.2" width="0.3048" layer="1"/>
+<wire x1="47.8" y1="10.6" x2="48.2" y2="10.2" width="0.4064" layer="1"/>
+<wire x1="61.8" y1="10.2" x2="61.8" y2="16.2" width="0.3048" layer="16"/>
+<wire x1="50.4" y1="10.2" x2="50.4" y2="9.85" width="0.3048" layer="1"/>
+<wire x1="52.4" y1="46.4" x2="50.2" y2="48.6" width="0.3048" layer="1"/>
+<wire x1="60.8" y1="46.4" x2="52.4" y2="46.4" width="0.3048" layer="1"/>
+<wire x1="61.8" y1="45.4" x2="60.8" y2="46.4" width="0.3048" layer="1"/>
+<wire x1="61.8" y1="16.2" x2="61.8" y2="45.4" width="0.3048" layer="1"/>
+<via x="61.8" y="10.2" extent="1-16" drill="0.5"/>
+<via x="61.8" y="16.2" extent="1-16" drill="0.5"/>
+<wire x1="50.2" y1="48.6" x2="48.0926" y2="48.6" width="0.3048" layer="1"/>
+</signal>
 </signals>
