File: hardware/playa.sch (EAGLE design)
At the start: 89 parts, among them Q2 12.288MHz, Q3 8MHz, U1 ATMEGA328, U11 1.8v, U12 3.3v, U17 AVR_SPI_PRG_6PTH, U3 microSD Socket, U5 3.3v, U6 CN3083, U9 VS1053-L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

Commit message: modify battery voltage divider. it currently uses 35uA
Parts:
- R19: value 2M 1% -> 68k 1%
- R8: value 10M 1% -> 39k 1%
Changed lines of the file:
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@@
 <part name="U$3" library="tsop" deviceset="TSOP312X" device=""/>
 <part name="C11" library="rcl" deviceset="C-EU" device="C1206" value="4.7u"/>
-<part name="R8" library="rcl" deviceset="R-EU_" device="R0805W" value="10M 1%"/>
-<part name="R19" library="rcl" deviceset="R-EU_" device="R0805W" value="2M 1%"/>
+<part name="R8" library="rcl" deviceset="R-EU_" device="R0805W" value="39k 1%"/>
+<part name="R19" library="rcl" deviceset="R-EU_" device="R0805W" value="68k 1%"/>
 <part name="GND28" library="SparkFun" deviceset="GND" device=""/>
 <part name="C17" library="rcl" deviceset="C-EU" device="C0805" value="100nF"/>

Commit message: rename traces to match the names given in the source code
Connections:
- net O_DETECT renamed JACK_DETECT
- net VIN_DETECT renamed VBAT_DETECT
Changed lines of the file:
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@@
 <?xml version="1.0" encoding="utf-8"?>
 <!DOCTYPE eagle SYSTEM "eagle.dtd">
-<eagle version="6.1">
+<eagle version="6.4">
 <drawing>
 <settings>
@@
 </segment>
 </net>
-<net name="O_DETECT" class="0">
-<segment>
-<wire x1="208.28" y1="81.28" x2="226.06" y2="81.28" width="0.1524" layer="91"/>
-<label x="210.82" y="81.28" size="1.778" layer="95"/>
-<pinref part="U1" gate="G$1" pin="PC1(ADC1)"/>
-<pinref part="R24" gate="G$1" pin="1"/>
-</segment>
-<segment>
-<wire x1="347.98" y1="129.54" x2="355.6" y2="129.54" width="0.1524" layer="91"/>
-<label x="347.98" y="129.54" size="1.778" layer="95"/>
-<pinref part="X2" gate="G$1" pin="B"/>
-</segment>
-</net>
 <net name="N$17" class="0">
 <segment>
@@
 </segment>
 </net>
-<net name="VIN_DETECT" class="0">
+<net name="SW1" class="0">
+<segment>
+<wire x1="208.28" y1="73.66" x2="220.98" y2="73.66" width="0.1524" layer="91"/>
+<label x="210.82" y="73.66" size="1.778" layer="95"/>
+<pinref part="U1" gate="G$1" pin="PC4(ADC4/SDA)"/>
+</segment>
+<segment>
+<wire x1="309.88" y1="231.14" x2="309.88" y2="228.6" width="0.1524" layer="91"/>
+<wire x1="302.26" y1="231.14" x2="309.88" y2="231.14" width="0.1524" layer="91"/>
+<wire x1="309.88" y1="231.14" x2="309.88" y2="236.22" width="0.1524" layer="91"/>
+<junction x="309.88" y="231.14"/>
+<label x="302.26" y="231.14" size="1.778" layer="95"/>
+<pinref part="S1" gate="S" pin="2"/>
+<pinref part="R20" gate="G$1" pin="2"/>
+</segment>
+</net>
+<net name="SW2" class="0">
+<segment>
+<wire x1="327.66" y1="231.14" x2="327.66" y2="228.6" width="0.1524" layer="91"/>
+<wire x1="320.04" y1="231.14" x2="327.66" y2="231.14" width="0.1524" layer="91"/>
+<wire x1="327.66" y1="231.14" x2="327.66" y2="236.22" width="0.1524" layer="91"/>
+<junction x="327.66" y="231.14"/>
+<label x="320.04" y="231.14" size="1.778" layer="95"/>
+<pinref part="S2" gate="S" pin="2"/>
+<pinref part="R21" gate="G$1" pin="2"/>
+</segment>
+<segment>
+<wire x1="208.28" y1="76.2" x2="220.98" y2="76.2" width="0.1524" layer="91"/>
+<label x="210.82" y="76.2" size="1.778" layer="95"/>
+<pinref part="U1" gate="G$1" pin="PC3(ADC3)"/>
+</segment>
+</net>
+<net name="SW3" class="0">
+<segment>
+<wire x1="345.44" y1="231.14" x2="345.44" y2="228.6" width="0.1524" layer="91"/>
+<wire x1="337.82" y1="231.14" x2="345.44" y2="231.14" width="0.1524" layer="91"/>
+<wire x1="345.44" y1="231.14" x2="345.44" y2="236.22" width="0.1524" layer="91"/>
+<junction x="345.44" y="231.14"/>
+<label x="337.82" y="231.14" size="1.778" layer="95"/>
+<pinref part="S3" gate="S" pin="2"/>
+<pinref part="R22" gate="G$1" pin="2"/>
+</segment>
+<segment>
+<wire x1="208.28" y1="78.74" x2="220.98" y2="78.74" width="0.1524" layer="91"/>
+<label x="210.82" y="78.74" size="1.778" layer="95"/>
+<pinref part="U1" gate="G$1" pin="PC2(ADC2)"/>
+</segment>
+</net>
+<net name="JACK_DETECT" class="0">
+<segment>
+<wire x1="208.28" y1="81.28" x2="226.06" y2="81.28" width="0.1524" layer="91"/>
+<label x="210.82" y="81.28" size="1.778" layer="95"/>
+<pinref part="U1" gate="G$1" pin="PC1(ADC1)"/>
+<pinref part="R24" gate="G$1" pin="1"/>
+</segment>
+<segment>
+<wire x1="347.98" y1="129.54" x2="355.6" y2="129.54" width="0.1524" layer="91"/>
+<label x="347.98" y="129.54" size="1.778" layer="95"/>
+<pinref part="X2" gate="G$1" pin="B"/>
+</segment>
+</net>
+<net name="VBAT_DETECT" class="0">
+<segment>
+<wire x1="208.28" y1="71.12" x2="220.98" y2="71.12" width="0.1524" layer="91"/>
+<label x="210.82" y="71.12" size="1.778" layer="95"/>
+<pinref part="U1" gate="G$1" pin="PC5(ADC5/SCL)"/>
+</segment>
 <segment>
 <wire x1="7.62" y1="154.94" x2="7.62" y2="152.4" width="0.1524" layer="91"/>
@@
 <pinref part="C17" gate="G$1" pin="1"/>
 </segment>
-<segment>
-<wire x1="208.28" y1="71.12" x2="220.98" y2="71.12" width="0.1524" layer="91"/>
-<label x="210.82" y="71.12" size="1.778" layer="95"/>
-<pinref part="U1" gate="G$1" pin="PC5(ADC5/SCL)"/>
-</segment>
-</net>
-<net name="SW1" class="0">
-<segment>
-<wire x1="208.28" y1="73.66" x2="220.98" y2="73.66" width="0.1524" layer="91"/>
-<label x="210.82" y="73.66" size="1.778" layer="95"/>
-<pinref part="U1" gate="G$1" pin="PC4(ADC4/SDA)"/>
-</segment>
-<segment>
-<wire x1="309.88" y1="231.14" x2="309.88" y2="228.6" width="0.1524" layer="91"/>
-<wire x1="302.26" y1="231.14" x2="309.88" y2="231.14" width="0.1524" layer="91"/>
-<wire x1="309.88" y1="231.14" x2="309.88" y2="236.22" width="0.1524" layer="91"/>
-<junction x="309.88" y="231.14"/>
-<label x="302.26" y="231.14" size="1.778" layer="95"/>
-<pinref part="S1" gate="S" pin="2"/>
-<pinref part="R20" gate="G$1" pin="2"/>
-</segment>
-</net>
-<net name="SW2" class="0">
-<segment>
-<wire x1="327.66" y1="231.14" x2="327.66" y2="228.6" width="0.1524" layer="91"/>
-<wire x1="320.04" y1="231.14" x2="327.66" y2="231.14" width="0.1524" layer="91"/>
-<wire x1="327.66" y1="231.14" x2="327.66" y2="236.22" width="0.1524" layer="91"/>
-<junction x="327.66" y="231.14"/>
-<label x="320.04" y="231.14" size="1.778" layer="95"/>
-<pinref part="S2" gate="S" pin="2"/>
-<pinref part="R21" gate="G$1" pin="2"/>
-</segment>
-<segment>
-<wire x1="208.28" y1="76.2" x2="220.98" y2="76.2" width="0.1524" layer="91"/>
-<label x="210.82" y="76.2" size="1.778" layer="95"/>
-<pinref part="U1" gate="G$1" pin="PC3(ADC3)"/>
-</segment>
-</net>
-<net name="SW3" class="0">
-<segment>
-<wire x1="345.44" y1="231.14" x2="345.44" y2="228.6" width="0.1524" layer="91"/>
-<wire x1="337.82" y1="231.14" x2="345.44" y2="231.14" width="0.1524" layer="91"/>
-<wire x1="345.44" y1="231.14" x2="345.44" y2="236.22" width="0.1524" layer="91"/>
-<junction x="345.44" y="231.14"/>
-<label x="337.82" y="231.14" size="1.778" layer="95"/>
-<pinref part="S3" gate="S" pin="2"/>
-<pinref part="R22" gate="G$1" pin="2"/>
-</segment>
-<segment>
-<wire x1="208.28" y1="78.74" x2="220.98" y2="78.74" width="0.1524" layer="91"/>
-<label x="210.82" y="78.74" size="1.778" layer="95"/>
-<pinref part="U1" gate="G$1" pin="PC2(ADC2)"/>
-</segment>
-</net>
+</net>
